Commit message: Added config file for 4 wheel drive and made necessary changes in the urdf files. The odom is consistently moving away from robot, so need to fix that.

File: urdf/robot.urdf.xacro (robot description, xacro)
@@ -1,8 +1,9 @@
 <?xml version="1.0" ?>
 <!-- =================================================================================== -->
-<!-- |    This document was autogenerated by xacro from urdf/wrv4/wrv4.xacro           | -->
+<!-- |    This document was autogenerated by xacro from urdf/robot.xacro               | -->
 <!-- |    EDITING THIS FILE BY HAND IS NOT RECOMMENDED                                 | -->
 <!-- =================================================================================== -->
-<robot name="wrv4">
+<robot name="wrv4" xmlns:xacro="http://www.ros.org/wiki/xacro">
+  <xacro:arg name="four_wheel_drive" default="$(find wheel_robot_v4)/config/four_wheel_diff_drive.yaml" />
   <material name="pet">
     <color rgba="0.700 0.700 0.700 1.000"/>
@@ -177,5 +178,5 @@
   </joint>
   <joint name="wheelfl_joint" type="continuous">
-    <origin rpy="-1.571 0 0" xyz="0.1 0.1125 -0.0375"/>
+    <origin rpy="1.571 0 0" xyz="0.1 0.1125 -0.0375"/>
     <parent link="base_link"/>
     <child link="wheelfl_link"/>
@@ -183,5 +184,5 @@
   </joint>
   <joint name="wheelfr_joint" type="continuous">
-    <origin rpy="-1.571 0 0" xyz="0.1 -0.1125 -0.0375"/>
+    <origin rpy="1.571 0 0" xyz="0.1 -0.1125 -0.0375"/>
     <parent link="base_link"/>
     <child link="wheelfr_link"/>
@@ -231,11 +232,11 @@
   <gazebo reference="wheelbl_link">
     <material>Gazebo/Yellow</material>
-    <mu1 value="0.01"/>
-    <mu2 value="0.01"/>
+    <!-- <mu1 value="0.01"/>
+  <mu2 value="0.01"/> -->
   </gazebo>
   <gazebo reference="wheelbr_link">
     <material>Gazebo/Yellow</material>
-    <mu1 value="0.01"/>
-    <mu2 value="0.01"/>
+    <!-- <mu1 value="0.01"/>
+  <mu2 value="0.01"/> -->
   </gazebo>
   <gazebo reference="camera_link">
@@ -315,5 +316,5 @@
       </plugin>
       <always_on>true</always_on>
-      <update_rate>30</update_rate>
+      <update_rate>100</update_rate>
       <visualize>true</visualize>
       <imu>
@@ -373,43 +374,73 @@
     </sensor>
   </gazebo>
+  <!-- <gazebo>
+  <plugin name='wrv4_diff_drive' filename='libgazebo_ros_diff_drive.so'>
+    <update_rate>30</update_rate>
+    <left_joint>wheelfl_joint</left_joint>
+    <right_joint>wheelfr_joint</right_joint>
+    <wheel_separation>0.2</wheel_separation>
+    <wheel_diameter>0.1</wheel_diameter>
+    <max_wheel_torque>20</max_wheel_torque>
+    <max_wheel_acceleration>1.0</max_wheel_acceleration>
+    <command_topic>cmd_vel</command_topic>
+    <publish_odom>true</publish_odom>
+    <publish_odom_tf>true</publish_odom_tf>
+    <publish_wheel_tf>false</publish_wheel_tf>
+    <odometry_topic>odom</odometry_topic>
+    <odometry_frame>odom</odometry_frame>
+    <robot_base_frame>base_footprint</robot_base_frame>
+  </plugin>
+</gazebo>
+<gazebo>
+  <plugin name="wrv4_joint_state" filename="libgazebo_ros_joint_state_publisher.so">
+    <ros>
+      <remapping>~/out:=joint_states</remapping>
+    </ros>
+    <update_rate>30</update_rate>
+    <joint_name>wheelfl_joint</joint_name>
+    <joint_name>wheelfr_joint</joint_name>
+  </plugin>
+</gazebo> -->
+  <ros2_control name="GazeboSystem" type="system">
+    <hardware>
+      <plugin>gazebo_ros2_control/GazeboSystem</plugin>
+    </hardware>
+    <joint name="wheelfl_joint">
+      <command_interface name="velocity">
+        <param name="min">-1</param>
+        <param name="max">1</param>
+      </command_interface>
+      <state_interface name="position"/>
+      <state_interface name="velocity"/>
+    </joint>
+    <joint name="wheelfr_joint">
+      <command_interface name="velocity">
+        <param name="min">-1</param>
+        <param name="max">1</param>
+      </command_interface>
+      <state_interface name="position"/>
+      <state_interface name="velocity"/>
+    </joint>
+    <joint name="wheelbl_joint">
+      <command_interface name="velocity">
+        <param name="min">-1</param>
+        <param name="max">1</param>
+      </command_interface>
+      <state_interface name="position"/>
+      <state_interface name="velocity"/>
+    </joint>
+    <joint name="wheelbr_joint">
+      <command_interface name="velocity">
+        <param name="min">-1</param>
+        <param name="max">1</param>
+      </command_interface>
+      <state_interface name="position"/>
+      <state_interface name="velocity"/>
+    </joint>
+  </ros2_control>
   <gazebo>
-    <plugin filename="libgazebo_ros_diff_drive.so" name="wrv4_diff_drive">
-      <ros>
-        <!--<namespace>/wrv3</namespace>-->
-      </ros>
-      <update_rate>30</update_rate>
-      <!-- wheels -->
-      <left_joint>wheelfl_joint</left_joint>
-      <!-- <left_joint>wheel2l_joint</left_joint> -->
-      <right_joint>wheelfr_joint</right_joint>
-      <!-- <right_joint>wheel2r_joint</right_joint> -->
-      <!-- kinematics -->
-      <wheel_separation>0.2</wheel_separation>
-      <wheel_diameter>0.1</wheel_diameter>
-      <!-- limits -->
-      <max_wheel_torque>20</max_wheel_torque>
-      <max_wheel_acceleration>1.0</max_wheel_acceleration>
-      <command_topic>cmd_vel</command_topic>
-      <!-- output -->
-      <publish_odom>true</publish_odom>
-      <publish_odom_tf>true</publish_odom_tf>
-      <publish_wheel_tf>false</publish_wheel_tf>
-      <odometry_topic>odom</odometry_topic>
-      <odometry_frame>odom</odometry_frame>
-      <robot_base_frame>base_footprint</robot_base_frame>
+    <plugin filename="libgazebo_ros2_control.so" name="gazebo_ros2_control">
+      <parameters>$(arg four_wheel_drive)</parameters>
     </plugin>
   </gazebo>
-  <gazebo>
-    <plugin filename="libgazebo_ros_joint_state_publisher.so" name="wrv4_joint_state">
-      <ros>
-        <!-- <namespace>/wrv3</namespace> -->
-        <remapping>~/out:=joint_states</remapping>
-      </ros>
-      <update_rate>30</update_rate>
-      <joint_name>wheelfl_joint</joint_name>
-      <!-- <joint_name>wheel2l_joint</joint_name> -->
-      <joint_name>wheelfr_joint</joint_name>
-      <!-- <joint_name>wheel2r_joint</joint_name> -->
-    </plugin>
-  </gazebo>
 </robot>

File: urdf/robot.xacro (robot description, xacro)
@@ -154,5 +154,5 @@
     </joint>
     <joint name="wheelfl_joint" type="continuous">
-        <origin xyz="0.1 0.1125 -0.0375" rpy="-1.571 0 0"/>
+        <origin xyz="0.1 0.1125 -0.0375" rpy="1.571 0 0"/>
         <parent link="base_link"/>
         <child link="wheelfl_link"/>
@@ -160,5 +160,5 @@
     </joint>
     <joint name="wheelfr_joint" type="continuous">
-        <origin xyz="0.1 -0.1125 -0.0375" rpy="-1.571 0 0"/>
+        <origin xyz="0.1 -0.1125 -0.0375" rpy="1.571 0 0"/>
         <parent link="base_link"/>
         <child link="wheelfr_link"/>

Commit message: Changes done to accomodate ros2_control DiffDriveController for 4 wheel drive. The Transform tree works well now. But while turning, the robot in gazebo doesn't rotate. Need to fix that.

File: urdf/robot.urdf.xacro (robot description, xacro)
@@ -178,5 +178,5 @@
   </joint>
   <joint name="wheelfl_joint" type="continuous">
-    <origin rpy="1.571 0 0" xyz="0.1 0.1125 -0.0375"/>
+    <origin rpy="-1.571 0 0" xyz="0.1 0.1125 -0.0375"/>
     <parent link="base_link"/>
     <child link="wheelfl_link"/>
@@ -184,5 +184,5 @@
   </joint>
   <joint name="wheelfr_joint" type="continuous">
-    <origin rpy="1.571 0 0" xyz="0.1 -0.1125 -0.0375"/>
+    <origin rpy="-1.571 0 0" xyz="0.1 -0.1125 -0.0375"/>
     <parent link="base_link"/>
     <child link="wheelfr_link"/>
@@ -190,5 +190,5 @@
   </joint>
   <joint name="wheelbl_joint" type="continuous">
-    <origin rpy="1.571 0 0" xyz="-0.1 0.1125 -0.0375"/>
+    <origin rpy="-1.571 0 0" xyz="-0.1 0.1125 -0.0375"/>
     <parent link="base_link"/>
     <child link="wheelbl_link"/>
@@ -196,5 +196,5 @@
   </joint>
   <joint name="wheelbr_joint" type="continuous">
-    <origin rpy="1.571 0 0" xyz="-0.1 -0.1125 -0.0375"/>
+    <origin rpy="-1.571 0 0" xyz="-0.1 -0.1125 -0.0375"/>
     <parent link="base_link"/>
     <child link="wheelbr_link"/>
@@ -442,4 +442,8 @@
     <plugin filename="libgazebo_ros2_control.so" name="gazebo_ros2_control">
       <parameters>$(arg four_wheel_drive)</parameters>
+      <ros>
+        <remapping>~/cmd_vel_unstamped:=/cmd_vel</remapping>
+        <remapping>~/odom:=/odom</remapping>
+      </ros>
     </plugin>
   </gazebo>

File: urdf/robot.xacro (robot description, xacro)
@@ -154,5 +154,5 @@
     </joint>
     <joint name="wheelfl_joint" type="continuous">
-        <origin xyz="0.1 0.1125 -0.0375" rpy="1.571 0 0"/>
+        <origin xyz="0.1 0.1125 -0.0375" rpy="-1.571 0 0"/>
         <parent link="base_link"/>
         <child link="wheelfl_link"/>
@@ -160,5 +160,5 @@
     </joint>
     <joint name="wheelfr_joint" type="continuous">
-        <origin xyz="0.1 -0.1125 -0.0375" rpy="1.571 0 0"/>
+        <origin xyz="0.1 -0.1125 -0.0375" rpy="-1.571 0 0"/>
         <parent link="base_link"/>
         <child link="wheelfr_link"/>
@@ -166,5 +166,5 @@
     </joint>
     <joint name="wheelbl_joint" type="continuous">
-        <origin xyz="-0.1 0.1125 -0.0375" rpy="1.571 0 0"/>
+        <origin xyz="-0.1 0.1125 -0.0375" rpy="-1.571 0 0"/>
         <parent link="base_link"/>
         <child link="wheelbl_link"/>
@@ -172,5 +172,5 @@
     </joint>
     <joint name="wheelbr_joint" type="continuous">
-        <origin xyz="-0.1 -0.1125 -0.0375" rpy="1.571 0 0"/>
+        <origin xyz="-0.1 -0.1125 -0.0375" rpy="-1.571 0 0"/>
         <parent link="base_link"/>
         <child link="wheelbr_link"/>
